File: waveshare_usb3300_to_dual_pmod.kicad_sch (KiCad schematic)
At the start: 4 parts, among them J1 Conn_01x02_Pin, J2 PMOD, J3 PMOD, J4 Conn_02x10_Top_Bottom

Commit message: waveshare_usb3300_to_dual_pmod: changed j4 footprint, resize PCB
Parts:
- J4: footprint Connector_PinHeader_2.54mm:PinHeader_2x10_P2.54mm_Vertical -> usb3300_connector:PinSocket_2x10_P2.54mm_Horizontal
Changed lines of the file:
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@@
 			)
 		)
-		(property "Footprint" "Connector_PinHeader_2.54mm:PinHeader_2x10_P2.54mm_Vertical"
+		(property "Footprint" "usb3300_connector:PinSocket_2x10_P2.54mm_Horizontal"
 			(at 177.8 88.9 0)
 			(hide yes)
